Commit message: feat: integrate realsense2_description and update URDF for omy_f3m arm

File: open_manipulator_description/urdf/omy_f3m/omy_f3m_arm.urdf.xacro (robot description, xacro)
@@ -2,4 +2,5 @@
 <robot xmlns:xacro="http://www.ros.org/wiki/xacro">
    <xacro:macro name="omy_f3m" params="prefix">
+      <xacro:include filename="$(find realsense2_description)/urdf/_d405.urdf.xacro" />
       <xacro:property name="meshes_file_direction" value="package://open_manipulator_description/meshes/omy_f3m" />
       <link name="${prefix}link0">
@@ -187,5 +188,5 @@
             <origin xyz="0 0 0" rpy="0 0 0" />
             <geometry>
-               <mesh filename="${meshes_file_direction}/link6.stl" scale="0.001 0.001 0.001" />
+               <mesh filename="${meshes_file_direction}/end_unit.stl" scale="0.001 0.001 0.001" />
             </geometry>
             <material name="grey">
@@ -205,4 +206,7 @@
          </inertial>
       </link>
+      <xacro:sensor_d405 parent="${prefix}link6" use_nominal_extrinsics="false" name="${prefix}camera">
+         <origin xyz="-0.021 -0.07385 0.0803" rpy="-1.57079632679 0 -1.57079632679"/>
+      </xacro:sensor_d405>
       <joint name="${prefix}end_effector_flange_joint" type="fixed">
          <parent link="${prefix}link6" />

Commit message: fix: update mesh filename in omy_f3m arm URDF from end_unit.stl to link6.stl

File: open_manipulator_description/urdf/omy_f3m/omy_f3m_arm.urdf.xacro (robot description, xacro)
@@ -188,5 +188,5 @@
             <origin xyz="0 0 0" rpy="0 0 0" />
             <geometry>
-               <mesh filename="${meshes_file_direction}/end_unit.stl" scale="0.001 0.001 0.001" />
+               <mesh filename="${meshes_file_direction}/link6.stl" scale="0.001 0.001 0.001" />
             </geometry>
             <material name="grey">
